Commit message: added prefix/namespace possibility to mir_description

File: mir_description/urdf/include/mir_100_v1.urdf.xacro (robot description, xacro)
@@ -24,5 +24,5 @@
   <xacro:property name="mir_100_caster_wheel_base_dz" value="${mir_100_caster_wheel_radius-mir_100_caster_wheel_dz}" />
   <xacro:property name="imu_stdev" value="0.00017" />
-  <xacro:macro name="actuated_wheel" params="prefix locationprefix locationright">
+  <xacro:macro name="actuated_wheel" params="prefix namespace locationprefix locationright">
     <joint name="${prefix}${locationprefix}_wheel_joint" type="continuous">
       <origin xyz="0.0 ${-mir_100_act_wheel_dy * locationright} ${mir_100_act_wheel_radius}" rpy="0 0 0" />
@@ -64,5 +64,7 @@
     </joint>
     <gazebo>
-      <plugin name="joint_states" filename="libgazebo_ros_joint_state_publisher.so">
+      <plugin name="${locationprefix}_caster_rotation_joint_states" filename="libgazebo_ros_joint_state_publisher.so">
+        <ros>
+        </ros>
         <update_rate>200.0</update_rate>
         <joint_name>${prefix}${locationprefix}_caster_rotation_joint</joint_name>
@@ -107,5 +109,8 @@
     </joint>
     <gazebo>
-      <plugin name="joint_states" filename="libgazebo_ros_joint_state_publisher.so">
+      <plugin name="${locationprefix}_caster_wheel_joint_states" filename="libgazebo_ros_joint_state_publisher.so">
+        <ros>
+          <namespace>${namespace}</namespace>
+        </ros>
         <update_rate>200.0</update_rate>
         <joint_name>${prefix}${locationprefix}_caster_wheel_joint</joint_name>
@@ -134,5 +139,5 @@
     </gazebo>
   </xacro:macro>
-  <xacro:macro name="mir_100" params="prefix">
+  <xacro:macro name="mir_100" params="prefix namespace">
     <link name="${prefix}base_footprint" />
     <joint name="${prefix}base_joint" type="fixed">
@@ -169,5 +174,5 @@
     </joint>
     <link name="${prefix}imu_link" />
-    <xacro:imu_gazebo link="${prefix}imu_link" imu_topic="imu_data" update_rate="50.0" stdev="${imu_stdev}" />
+    <xacro:imu_gazebo link="${prefix}imu_link" imu_topic="${prefix}imu_data" update_rate="50.0" stdev="${imu_stdev}" />
     <!-- Create an alias for imu_link. This is necessary because the real MiR's
          TF has imu_link, but the imu_data topic is published in the imu_frame
@@ -185,5 +190,5 @@
       <origin xyz="0.4288 0.2358 0.1914" rpy="0.0 0.0 ${0.25 * pi}" />  <!-- from visually matching up the meshes of the MiR and the laser scanner -->
     </joint>
-    <xacro:sick_s300 prefix="${prefix}" link="front_laser_link" topic="f_scan" />
+    <xacro:sick_s300 prefix="${prefix}" namespace="${namespace}" link="front_laser_link" topic="f_scan" />
     <joint name="${prefix}base_link_to_back_laser_joint" type="fixed">
       <parent link="${prefix}base_link" />
@@ -191,5 +196,5 @@
       <origin xyz="-0.3548 -0.2352 0.1914" rpy="0.0 0.0 ${-0.75 * pi}" />  <!-- from visually matching up the meshes of the MiR and the laser scanner -->
     </joint>
-    <xacro:sick_s300 prefix="${prefix}" link="back_laser_link" topic="b_scan" />
+    <xacro:sick_s300 prefix="${prefix}" namespace="${namespace}" link="back_laser_link" topic="b_scan" />
     <!-- Ultrasound sensors -->
     <joint name="${prefix}us_1_joint" type="fixed">   <!-- right ultrasound -->
@@ -206,6 +211,6 @@
     <link name="${prefix}us_2_frame" />
     <!-- wheels -->
-    <xacro:actuated_wheel prefix="${prefix}" locationprefix="left" locationright="-1"/>
-    <xacro:actuated_wheel prefix="${prefix}" locationprefix="right" locationright="1"/>
+    <xacro:actuated_wheel prefix="${prefix}" namespace="${namespace}" locationprefix="left" locationright="-1"/>
+    <xacro:actuated_wheel prefix="${prefix}" namespace="${namespace}" locationprefix="right" locationright="1"/>
     <xacro:caster_wheel prefix="${prefix}" locationprefix="fl" locationright="-1" wheel_base_dx="${mir_100_front_caster_wheel_base_dx}"/>
     <xacro:caster_wheel prefix="${prefix}" locationprefix="fr" locationright="1" wheel_base_dx="${mir_100_front_caster_wheel_base_dx}"/>
@@ -222,5 +227,5 @@
     <!-- set the gazebo friction parameters for the wheels -->
     <xacro:set_all_wheel_frictions prefix="${prefix}"/>
-    <xacro:p3d_base_controller prefix="${prefix}" />
+    <xacro:p3d_base_controller prefix="${prefix}" namespace="${namespace}"/>
   </xacro:macro>
 </robot>

File: mir_description/urdf/include/sick_s300.urdf.xacro (robot description, xacro)
@@ -6,5 +6,5 @@
   <xacro:property name="laser_z" value="0.185" />
   <xacro:property name="laser_mass" value="2.0" />
-  <xacro:macro name="sick_s300" params="link topic prefix">
+  <xacro:macro name="sick_s300" params="link topic prefix namespace">
     <link name="${prefix}${link}">
       <visual>
@@ -58,4 +58,5 @@
           <ros>
             <remapping>~/out:=${topic}</remapping>
+            <namespace>${namespace}</namespace>
           </ros>
           <output_type>sensor_msgs/LaserScan</output_type>

Commit message: Add namespace support
* add namespace for simulation and teleop

* add namespace to gazebo entity

* change to prefix only in urdfs

* enable ns for joint_state_publisher

* add namespace support to mir_navigation + ns instructions to readme

* switched namespaces to remappings in urdfs

* resolved gazeboplugin namespace errors

* fixes for namespace support driver

* added navigation config namespace examples

* minor fixes for namespace launch and adaptions in rviz configs

* fixed tf namespace bug in driver

* split up of driver launch files

* fixed params filename + added namespace args in nav launch

* enabled qos settings for ros2 topics in driver

* removed unused rviz parameter

See relffok/mir_robot#17

File: mir_description/urdf/include/mir_100_v1.urdf.xacro (robot description, xacro)
@@ -24,5 +24,5 @@
   <xacro:property name="mir_100_caster_wheel_base_dz" value="${mir_100_caster_wheel_radius-mir_100_caster_wheel_dz}" />
   <xacro:property name="imu_stdev" value="0.00017" />
-  <xacro:macro name="actuated_wheel" params="prefix namespace locationprefix locationright">
+  <xacro:macro name="actuated_wheel" params="prefix locationprefix locationright">
     <joint name="${prefix}${locationprefix}_wheel_joint" type="continuous">
       <origin xyz="0.0 ${-mir_100_act_wheel_dy * locationright} ${mir_100_act_wheel_radius}" rpy="0 0 0" />
@@ -54,5 +54,5 @@
     </gazebo>
   </xacro:macro>
-  <xacro:macro name="caster_wheel" params="prefix locationprefix locationright wheel_base_dx">
+  <xacro:macro name="caster_wheel" params="prefix ns locationprefix locationright wheel_base_dx">
     <!-- caster hub -->
     <joint name="${prefix}${locationprefix}_caster_rotation_joint" type="continuous">
@@ -66,4 +66,5 @@
       <plugin name="${locationprefix}_caster_rotation_joint_states" filename="libgazebo_ros_joint_state_publisher.so">
         <ros>
+          <namespace>${ns}</namespace>
         </ros>
         <update_rate>200.0</update_rate>
@@ -111,5 +112,5 @@
       <plugin name="${locationprefix}_caster_wheel_joint_states" filename="libgazebo_ros_joint_state_publisher.so">
         <ros>
-          <namespace>${namespace}</namespace>
+          <namespace>${ns}</namespace>
         </ros>
         <update_rate>200.0</update_rate>
@@ -139,5 +140,5 @@
     </gazebo>
   </xacro:macro>
-  <xacro:macro name="mir_100" params="prefix namespace">
+  <xacro:macro name="mir_100" params="prefix ns">
     <link name="${prefix}base_footprint" />
     <joint name="${prefix}base_joint" type="fixed">
@@ -198,5 +199,5 @@
       <origin xyz="0.4288 0.2358 0.1914" rpy="0.0 0.0 ${0.25 * pi}" />  <!-- from visually matching up the meshes of the MiR and the laser scanner -->
     </joint>
-    <xacro:sick_s300 prefix="${prefix}" namespace="${namespace}" link="front_laser_link" topic="f_scan" />
+    <xacro:sick_s300 prefix="${prefix}" link="front_laser_link" topic="f_scan" />
     <joint name="${prefix}base_link_to_back_laser_joint" type="fixed">
       <parent link="${prefix}base_link" />
@@ -204,5 +205,5 @@
       <origin xyz="-0.3548 -0.2352 0.1914" rpy="0.0 0.0 ${-0.75 * pi}" />  <!-- from visually matching up the meshes of the MiR and the laser scanner -->
     </joint>
-    <xacro:sick_s300 prefix="${prefix}" namespace="${namespace}" link="back_laser_link" topic="b_scan" />
+    <xacro:sick_s300 prefix="${prefix}" link="back_laser_link" topic="b_scan" />
     <!-- Ultrasound sensors -->
     <joint name="${prefix}us_1_joint" type="fixed">   <!-- right ultrasound -->
@@ -219,10 +220,10 @@
     <link name="${prefix}us_2_frame" />
     <!-- wheels -->
-    <xacro:actuated_wheel prefix="${prefix}" namespace="${namespace}" locationprefix="left" locationright="-1"/>
-    <xacro:actuated_wheel prefix="${prefix}" namespace="${namespace}" locationprefix="right" locationright="1"/>
-    <xacro:caster_wheel prefix="${prefix}" locationprefix="fl" locationright="-1" wheel_base_dx="${mir_100_front_caster_wheel_base_dx}"/>
-    <xacro:caster_wheel prefix="${prefix}" locationprefix="fr" locationright="1" wheel_base_dx="${mir_100_front_caster_wheel_base_dx}"/>
-    <xacro:caster_wheel prefix="${prefix}" locationprefix="bl" locationright="-1" wheel_base_dx="${mir_100_back_caster_wheel_base_dx}"/>
-    <xacro:caster_wheel prefix="${prefix}" locationprefix="br" locationright="1" wheel_base_dx="${mir_100_back_caster_wheel_base_dx}"/>
+    <xacro:actuated_wheel prefix="${prefix}" locationprefix="left" locationright="-1"/>
+    <xacro:actuated_wheel prefix="${prefix}" locationprefix="right" locationright="1"/>
+    <xacro:caster_wheel prefix="${prefix}" ns="${ns}" locationprefix="fl" locationright="-1" wheel_base_dx="${mir_100_front_caster_wheel_base_dx}"/>
+    <xacro:caster_wheel prefix="${prefix}" ns="${ns}" locationprefix="fr" locationright="1" wheel_base_dx="${mir_100_front_caster_wheel_base_dx}"/>
+    <xacro:caster_wheel prefix="${prefix}" ns="${ns}" locationprefix="bl" locationright="-1" wheel_base_dx="${mir_100_back_caster_wheel_base_dx}"/>
+    <xacro:caster_wheel prefix="${prefix}" ns="${ns}" locationprefix="br" locationright="1" wheel_base_dx="${mir_100_back_caster_wheel_base_dx}"/>
     <joint name="${prefix}base_link_surface_joint" type="fixed">
       <origin xyz="${mir_100_act_wheel_dx} 0 0.352" rpy="0 0 0" />
@@ -235,5 +236,5 @@
     <!-- set the gazebo friction parameters for the wheels -->
     <xacro:set_all_wheel_frictions prefix="${prefix}"/>
-    <xacro:p3d_base_controller prefix="${prefix}" namespace="${namespace}"/>
+    <xacro:p3d_base_controller prefix="${prefix}" />
   </xacro:macro>
 </robot>

File: mir_description/urdf/include/sick_s300.urdf.xacro (robot description, xacro)
@@ -6,5 +6,5 @@
   <xacro:property name="laser_z" value="0.185" />
   <xacro:property name="laser_mass" value="2.0" />
-  <xacro:macro name="sick_s300" params="link topic prefix namespace">
+  <xacro:macro name="sick_s300" params="link topic prefix">
     <link name="${prefix}${link}">
       <visual>
@@ -57,6 +57,5 @@
         <plugin name="gazebo_ros_${link}_controller" filename="libgazebo_ros_ray_sensor.so">
           <ros>
-            <remapping>~/out:=${topic}</remapping>
-            <namespace>${namespace}</namespace>
+            <remapping>~/out:=${prefix}${topic}</remapping>
           </ros>
           <output_type>sensor_msgs/LaserScan</output_type>

Commit message: Refactor URDF to prepare for MiR250 support
* specify caster wheel dx, radius and width independent of active wheel
* use cylinder geometric primitive instead of mesh for visual tag of wheels
* pull out laser positions into properties

File: mir_description/urdf/include/mir_100_v1.urdf.xacro (robot description, xacro)
@@ -13,14 +13,18 @@
   <xacro:property name="mir_100_act_wheel_dx" value="0.037646" />
   <xacro:property name="mir_100_act_wheel_dy" value="0.222604" />
-  <xacro:property name="mir_100_caster_wheel_radius" value="${mir_100_act_wheel_radius}" />
-  <xacro:property name="mir_100_caster_wheel_width" value="${mir_100_act_wheel_width}" />
-  <xacro:property name="mir_100_caster_wheel_mass" value="${mir_100_act_wheel_mass}" />
+  <xacro:property name="mir_100_caster_wheel_radius" value="0.0625" />
+  <xacro:property name="mir_100_caster_wheel_width" value="0.032" />
+  <xacro:property name="mir_100_caster_wheel_mass" value="1.0" />
   <xacro:property name="mir_100_caster_wheel_dx" value="-0.0382" />
   <xacro:property name="mir_100_caster_wheel_dy" value="0" />
   <xacro:property name="mir_100_caster_wheel_dz" value="-0.094" />
-  <xacro:property name="mir_100_front_caster_wheel_base_dx" value="0.341346" />
-  <xacro:property name="mir_100_back_caster_wheel_base_dx" value="-0.270154" />
+  <xacro:property name="mir_100_front_caster_wheel_base_dx" value="0.3037" />
+  <xacro:property name="mir_100_back_caster_wheel_base_dx"  value="0.3078" />
   <xacro:property name="mir_100_caster_wheel_base_dy" value="0.203" />
-  <xacro:property name="mir_100_caster_wheel_base_dz" value="${mir_100_caster_wheel_radius-mir_100_caster_wheel_dz}" />
+  <xacro:property name="mir_100_caster_wheel_base_dz" value="${mir_100_caster_wheel_radius - mir_100_caster_wheel_dz}" />
+  <!-- from visually matching up the meshes of the MiR and the laser scanner -->
+  <xacro:property name="laser_dx" value="0.392" />
+  <xacro:property name="laser_dy" value="0.2358" />
+  <xacro:property name="laser_dz" value="0.1914" />
   <xacro:property name="imu_stdev" value="0.00017" />
   <xacro:macro name="actuated_wheel" params="prefix locationprefix locationright">
@@ -37,7 +41,7 @@
       </xacro:cylinder_inertial>
       <visual>
-        <origin xyz="0 0 0" rpy="0 0 0" />
-        <geometry>
-          <mesh filename="package://mir_description/meshes/visual/wheel.stl" />
+        <origin xyz="0 0 0" rpy="${pi/2} 0 0" />
+        <geometry>
+          <cylinder radius="${mir_100_act_wheel_radius}" length="${mir_100_act_wheel_width}" />
         </geometry>
         <xacro:insert_block name="material_dark_grey" />
@@ -123,7 +127,7 @@
       </xacro:cylinder_inertial>
       <visual>
-        <origin xyz="0 0 0" rpy="0 0 0" />
-        <geometry>
-          <mesh filename="package://mir_description/meshes/visual/wheel.stl" />
+        <origin xyz="0 0 0" rpy="${pi/2} 0 0" />
+        <geometry>
+          <cylinder radius="${mir_100_caster_wheel_radius}" length="${mir_100_caster_wheel_width}" />
         </geometry>
         <xacro:insert_block name="material_dark_grey" />
@@ -197,5 +201,5 @@
       <parent link="${prefix}base_link" />
       <child link="${prefix}front_laser_link" />
-      <origin xyz="0.4288 0.2358 0.1914" rpy="0.0 0.0 ${0.25 * pi}" />  <!-- from visually matching up the meshes of the MiR and the laser scanner -->
+      <origin xyz="${laser_dx + mir_100_act_wheel_dx} ${laser_dy} ${laser_dz}" rpy="0.0 0.0 ${0.25 * pi}" />
     </joint>
     <xacro:sick_s300 prefix="${prefix}" link="front_laser_link" topic="f_scan" />
@@ -203,5 +207,5 @@
       <parent link="${prefix}base_link" />
       <child link="${prefix}back_laser_link" />
-      <origin xyz="-0.3548 -0.2352 0.1914" rpy="0.0 0.0 ${-0.75 * pi}" />  <!-- from visually matching up the meshes of the MiR and the laser scanner -->
+      <origin xyz="${-laser_dx + mir_100_act_wheel_dx} ${-laser_dy} ${laser_dz}" rpy="0.0 0.0 ${-0.75 * pi}" />
     </joint>
     <xacro:sick_s300 prefix="${prefix}" link="back_laser_link" topic="b_scan" />
@@ -222,8 +226,8 @@
     <xacro:actuated_wheel prefix="${prefix}" locationprefix="left" locationright="-1"/>
     <xacro:actuated_wheel prefix="${prefix}" locationprefix="right" locationright="1"/>
-    <xacro:caster_wheel prefix="${prefix}" ns="${ns}" locationprefix="fl" locationright="-1" wheel_base_dx="${mir_100_front_caster_wheel_base_dx}"/>
-    <xacro:caster_wheel prefix="${prefix}" ns="${ns}" locationprefix="fr" locationright="1" wheel_base_dx="${mir_100_front_caster_wheel_base_dx}"/>
-    <xacro:caster_wheel prefix="${prefix}" ns="${ns}" locationprefix="bl" locationright="-1" wheel_base_dx="${mir_100_back_caster_wheel_base_dx}"/>
-    <xacro:caster_wheel prefix="${prefix}" ns="${ns}" locationprefix="br" locationright="1" wheel_base_dx="${mir_100_back_caster_wheel_base_dx}"/>
+    <xacro:caster_wheel prefix="${prefix}" ns="${ns}" locationprefix="fl" locationright="-1" wheel_base_dx="${mir_100_front_caster_wheel_base_dx + mir_100_act_wheel_dx}"/>
+    <xacro:caster_wheel prefix="${prefix}" ns="${ns}" locationprefix="fr" locationright="1" wheel_base_dx="${mir_100_front_caster_wheel_base_dx + mir_100_act_wheel_dx}"/>
+    <xacro:caster_wheel prefix="${prefix}" ns="${ns}" locationprefix="bl" locationright="-1" wheel_base_dx="${-mir_100_back_caster_wheel_base_dx + mir_100_act_wheel_dx}"/>
+    <xacro:caster_wheel prefix="${prefix}" ns="${ns}" locationprefix="br" locationright="1" wheel_base_dx="${-mir_100_back_caster_wheel_base_dx + mir_100_act_wheel_dx}"/>
     <joint name="${prefix}base_link_surface_joint" type="fixed">
       <origin xyz="${mir_100_act_wheel_dx} 0 0.352" rpy="0 0 0" />
