Commit message: Rename mir_100 -> mir
This is in preparation of mir_250 support.

sed -i 's/MiR100/MiR/g' $(git ls-files)
sed -i 's/MiR0/MiR1000/g' $(git ls-files)
sed -i 's/mir_100/mir/g' $(git ls-files)
sed -i 's/mir_base.stl/mir_100_base.stl/g' $(git ls-files)
cd  mir_description/urdf/include/
mmv mir_100* mir*

File: mir_description/urdf/include/mir_v1.urdf.xacro (robot description, xacro)
@@ -3,24 +3,24 @@
   <xacro:include filename="$(find mir_description)/urdf/include/common_properties.urdf.xacro" />
   <xacro:include filename="$(find mir_description)/urdf/include/imu.gazebo.urdf.xacro" />
-  <xacro:include filename="$(find mir_description)/urdf/include/mir_100.gazebo.xacro" />
-  <xacro:include filename="$(find mir_description)/urdf/include/mir_100.transmission.xacro" />
+  <xacro:include filename="$(find mir_description)/urdf/include/mir.gazebo.xacro" />
+  <xacro:include filename="$(find mir_description)/urdf/include/mir.transmission.xacro" />
   <xacro:include filename="$(find mir_description)/urdf/include/sick_s300.urdf.xacro" />
   <xacro:property name="deg_to_rad" value="0.017453293" />
-  <xacro:property name="mir_100_base_mass" value="58.0" />
-  <xacro:property name="mir_100_act_wheel_radius" value="0.0625" />
-  <xacro:property name="mir_100_act_wheel_width" value="0.032" />
-  <xacro:property name="mir_100_act_wheel_mass" value="1.0" />
-  <xacro:property name="mir_100_act_wheel_dx" value="0.037646" />
-  <xacro:property name="mir_100_act_wheel_dy" value="0.222604" />
-  <xacro:property name="mir_100_caster_wheel_radius" value="0.0625" />
-  <xacro:property name="mir_100_caster_wheel_width" value="0.032" />
-  <xacro:property name="mir_100_caster_wheel_mass" value="1.0" />
-  <xacro:property name="mir_100_caster_wheel_dx" value="-0.0382" />
-  <xacro:property name="mir_100_caster_wheel_dy" value="0" />
-  <xacro:property name="mir_100_caster_wheel_dz" value="-0.094" />
-  <xacro:property name="mir_100_front_caster_wheel_base_dx" value="0.3037" />
-  <xacro:property name="mir_100_back_caster_wheel_base_dx"  value="0.3078" />
-  <xacro:property name="mir_100_caster_wheel_base_dy" value="0.203" />
-  <xacro:property name="mir_100_caster_wheel_base_dz" value="${mir_100_caster_wheel_radius - mir_100_caster_wheel_dz}" />
+  <xacro:property name="mir_base_mass" value="58.0" />
+  <xacro:property name="mir_act_wheel_radius" value="0.0625" />
+  <xacro:property name="mir_act_wheel_width" value="0.032" />
+  <xacro:property name="mir_act_wheel_mass" value="1.0" />
+  <xacro:property name="mir_act_wheel_dx" value="0.037646" />
+  <xacro:property name="mir_act_wheel_dy" value="0.222604" />
+  <xacro:property name="mir_caster_wheel_radius" value="0.0625" />
+  <xacro:property name="mir_caster_wheel_width" value="0.032" />
+  <xacro:property name="mir_caster_wheel_mass" value="1.0" />
+  <xacro:property name="mir_caster_wheel_dx" value="-0.0382" />
+  <xacro:property name="mir_caster_wheel_dy" value="0" />
+  <xacro:property name="mir_caster_wheel_dz" value="-0.094" />
+  <xacro:property name="mir_front_caster_wheel_base_dx" value="0.3037" />
+  <xacro:property name="mir_back_caster_wheel_base_dx"  value="0.3078" />
+  <xacro:property name="mir_caster_wheel_base_dy" value="0.203" />
+  <xacro:property name="mir_caster_wheel_base_dz" value="${mir_caster_wheel_radius - mir_caster_wheel_dz}" />
   <!-- from visually matching up the meshes of the MiR and the laser scanner -->
   <xacro:property name="laser_dx" value="0.392" />
@@ -30,5 +30,5 @@
   <xacro:macro name="actuated_wheel" params="prefix locationprefix locationright">
     <joint name="${prefix}${locationprefix}_wheel_joint" type="continuous">
-      <origin xyz="0.0 ${-mir_100_act_wheel_dy * locationright} ${mir_100_act_wheel_radius}" rpy="0 0 0" />
+      <origin xyz="0.0 ${-mir_act_wheel_dy * locationright} ${mir_act_wheel_radius}" rpy="0 0 0" />
       <parent link="${prefix}base_link" />
       <child link="${prefix}${locationprefix}_wheel_link" />
@@ -37,5 +37,5 @@
     </joint>
     <link name="${prefix}${locationprefix}_wheel_link">
-      <xacro:cylinder_inertial mass="${mir_100_act_wheel_mass}" radius="${mir_100_act_wheel_radius}" length="${mir_100_act_wheel_width}">
+      <xacro:cylinder_inertial mass="${mir_act_wheel_mass}" radius="${mir_act_wheel_radius}" length="${mir_act_wheel_width}">
         <origin xyz="0 0 0" rpy="${0.5 * pi} 0 0" />
       </xacro:cylinder_inertial>
@@ -43,5 +43,5 @@
         <origin xyz="0 0 0" rpy="${pi/2} 0 0" />
         <geometry>
-          <cylinder radius="${mir_100_act_wheel_radius}" length="${mir_100_act_wheel_width}" />
+          <cylinder radius="${mir_act_wheel_radius}" length="${mir_act_wheel_width}" />
         </geometry>
         <xacro:insert_block name="material_dark_grey" />
@@ -50,5 +50,5 @@
         <origin xyz="0 0 0" rpy="${pi/2} 0 0" />
         <geometry>
-          <cylinder radius="${mir_100_act_wheel_radius}" length="${mir_100_act_wheel_width}" />
+          <cylinder radius="${mir_act_wheel_radius}" length="${mir_act_wheel_width}" />
         </geometry>
       </collision>
@@ -61,5 +61,5 @@
     <!-- caster hub -->
     <joint name="${prefix}${locationprefix}_caster_rotation_joint" type="continuous">
-      <origin xyz="${wheel_base_dx} ${-mir_100_caster_wheel_base_dy * locationright} ${mir_100_caster_wheel_base_dz}" rpy="0 0 0" />
+      <origin xyz="${wheel_base_dx} ${-mir_caster_wheel_base_dy * locationright} ${mir_caster_wheel_base_dz}" rpy="0 0 0" />
       <parent link="${prefix}base_link" />
       <child link="${prefix}${locationprefix}_caster_rotation_link" />
@@ -108,5 +108,5 @@
     <!-- caster wheel -->
     <joint name="${prefix}${locationprefix}_caster_wheel_joint" type="continuous">
-      <origin xyz="${mir_100_caster_wheel_dx} ${-mir_100_caster_wheel_dy * locationright} ${mir_100_caster_wheel_dz}" rpy="0 0 0" />
+      <origin xyz="${mir_caster_wheel_dx} ${-mir_caster_wheel_dy * locationright} ${mir_caster_wheel_dz}" rpy="0 0 0" />
       <parent link="${prefix}${locationprefix}_caster_rotation_link" />
       <child link="${prefix}${locationprefix}_caster_wheel_link" />
@@ -123,5 +123,5 @@
     </gazebo>
     <link name="${prefix}${locationprefix}_caster_wheel_link">
-      <xacro:cylinder_inertial mass="${mir_100_caster_wheel_mass}" radius="${mir_100_caster_wheel_radius}" length="${mir_100_caster_wheel_width}">
+      <xacro:cylinder_inertial mass="${mir_caster_wheel_mass}" radius="${mir_caster_wheel_radius}" length="${mir_caster_wheel_width}">
         <origin xyz="0 0 0" rpy="${0.5 * pi} 0 0" />
       </xacro:cylinder_inertial>
@@ -129,5 +129,5 @@
         <origin xyz="0 0 0" rpy="${pi/2} 0 0" />
         <geometry>
-          <cylinder radius="${mir_100_caster_wheel_radius}" length="${mir_100_caster_wheel_width}" />
+          <cylinder radius="${mir_caster_wheel_radius}" length="${mir_caster_wheel_width}" />
         </geometry>
         <xacro:insert_block name="material_dark_grey" />
@@ -136,5 +136,5 @@
         <origin xyz="0 0 0" rpy="${pi/2} 0 0" />
         <geometry>
-          <cylinder radius="${mir_100_caster_wheel_radius}" length="${mir_100_caster_wheel_width}" />
+          <cylinder radius="${mir_caster_wheel_radius}" length="${mir_caster_wheel_width}" />
         </geometry>
       </collision>
@@ -144,5 +144,5 @@
     </gazebo>
   </xacro:macro>
-  <xacro:macro name="mir_100" params="prefix ns">
+  <xacro:macro name="mir" params="prefix ns">
     <link name="${prefix}base_footprint" />
     <joint name="${prefix}base_joint" type="fixed">
@@ -152,9 +152,9 @@
     </joint>
     <link name="${prefix}base_link">
-      <xacro:box_inertial mass="${mir_100_base_mass}" x="0.9" y="0.58" z="0.3">
-        <origin xyz="${mir_100_act_wheel_dx} 0 0.20" rpy="0 0 0" />
+      <xacro:box_inertial mass="${mir_base_mass}" x="0.9" y="0.58" z="0.3">
+        <origin xyz="${mir_act_wheel_dx} 0 0.20" rpy="0 0 0" />
       </xacro:box_inertial>
       <visual>
-        <origin xyz="${mir_100_act_wheel_dx} 0 0" rpy="0 0 0" />
+        <origin xyz="${mir_act_wheel_dx} 0 0" rpy="0 0 0" />
         <geometry>
           <mesh filename="package://mir_description/meshes/visual/mir_100_base.stl" />
@@ -163,5 +163,5 @@
       </visual>
       <collision>
-        <origin xyz="${mir_100_act_wheel_dx} 0 0" rpy="0 0 0" />
+        <origin xyz="${mir_act_wheel_dx} 0 0" rpy="0 0 0" />
         <geometry>
           <mesh filename="package://mir_description/meshes/collision/mir_100_base.stl" />
@@ -201,5 +201,5 @@
       <parent link="${prefix}base_link" />
       <child link="${prefix}front_laser_link" />
-      <origin xyz="${laser_dx + mir_100_act_wheel_dx} ${laser_dy} ${laser_dz}" rpy="0.0 0.0 ${0.25 * pi}" />
+      <origin xyz="${laser_dx + mir_act_wheel_dx} ${laser_dy} ${laser_dz}" rpy="0.0 0.0 ${0.25 * pi}" />
     </joint>
     <xacro:sick_s300 prefix="${prefix}" link="front_laser_link" topic="f_scan" />
@@ -207,5 +207,5 @@
       <parent link="${prefix}base_link" />
       <child link="${prefix}back_laser_link" />
-      <origin xyz="${-laser_dx + mir_100_act_wheel_dx} ${-laser_dy} ${laser_dz}" rpy="0.0 0.0 ${-0.75 * pi}" />
+      <origin xyz="${-laser_dx + mir_act_wheel_dx} ${-laser_dy} ${laser_dz}" rpy="0.0 0.0 ${-0.75 * pi}" />
     </joint>
     <xacro:sick_s300 prefix="${prefix}" link="back_laser_link" topic="b_scan" />
@@ -226,10 +226,10 @@
     <xacro:actuated_wheel prefix="${prefix}" locationprefix="left" locationright="-1"/>
     <xacro:actuated_wheel prefix="${prefix}" locationprefix="right" locationright="1"/>
-    <xacro:caster_wheel prefix="${prefix}" ns="${ns}" locationprefix="fl" locationright="-1" wheel_base_dx="${mir_100_front_caster_wheel_base_dx + mir_100_act_wheel_dx}"/>
-    <xacro:caster_wheel prefix="${prefix}" ns="${ns}" locationprefix="fr" locationright="1" wheel_base_dx="${mir_100_front_caster_wheel_base_dx + mir_100_act_wheel_dx}"/>
-    <xacro:caster_wheel prefix="${prefix}" ns="${ns}" locationprefix="bl" locationright="-1" wheel_base_dx="${-mir_100_back_caster_wheel_base_dx + mir_100_act_wheel_dx}"/>
-    <xacro:caster_wheel prefix="${prefix}" ns="${ns}" locationprefix="br" locationright="1" wheel_base_dx="${-mir_100_back_caster_wheel_base_dx + mir_100_act_wheel_dx}"/>
+    <xacro:caster_wheel prefix="${prefix}" ns="${ns}" locationprefix="fl" locationright="-1" wheel_base_dx="${mir_front_caster_wheel_base_dx + mir_act_wheel_dx}"/>
+    <xacro:caster_wheel prefix="${prefix}" ns="${ns}" locationprefix="fr" locationright="1" wheel_base_dx="${mir_front_caster_wheel_base_dx + mir_act_wheel_dx}"/>
+    <xacro:caster_wheel prefix="${prefix}" ns="${ns}" locationprefix="bl" locationright="-1" wheel_base_dx="${-mir_back_caster_wheel_base_dx + mir_act_wheel_dx}"/>
+    <xacro:caster_wheel prefix="${prefix}" ns="${ns}" locationprefix="br" locationright="1" wheel_base_dx="${-mir_back_caster_wheel_base_dx + mir_act_wheel_dx}"/>
     <joint name="${prefix}base_link_surface_joint" type="fixed">
-      <origin xyz="${mir_100_act_wheel_dx} 0 0.352" rpy="0 0 0" />
+      <origin xyz="${mir_act_wheel_dx} 0 0.352" rpy="0 0 0" />
       <parent link="${prefix}base_link" />
       <child link="${prefix}surface" />
@@ -237,5 +237,5 @@
     </joint>
     <link name="${prefix}surface"/>
-    <xacro:mir_100_wheel_transmissions prefix="${prefix}"/>
+    <xacro:mir_wheel_transmissions prefix="${prefix}"/>
     <!-- set the gazebo friction parameters for the wheels -->
     <xacro:set_all_wheel_frictions prefix="${prefix}"/>

File: mir_description/urdf/mir.urdf.xacro (robot description, xacro)
@@ -1,9 +1,9 @@
 <?xml version="1.0"?>
 <robot xmlns:xacro="http://ros.org/wiki/xacro"
-       name="mir_100" >
-  <!-- MiR100 base -->
-  <xacro:include filename="$(find mir_description)/urdf/include/mir_100_v1.urdf.xacro" />
+       name="mir" >
+  <!-- MiR base -->
+  <xacro:include filename="$(find mir_description)/urdf/include/mir_v1.urdf.xacro" />
   <xacro:include filename="$(find mir_description)/urdf/include/common.gazebo.xacro" />
-  <xacro:include filename="$(find mir_description)/urdf/include/mir_100.gazebo.xacro" />
+  <xacro:include filename="$(find mir_description)/urdf/include/mir.gazebo.xacro" />
   <xacro:arg name="tf_prefix" default="" />
   <!-- prefix can not start with a slash like a global namespace! results in TF errors -->
@@ -15,9 +15,9 @@
     <xacro:property name="prefix" value="${ns}/" />
   </xacro:unless>
-  <xacro:mir_100 prefix="${prefix}" ns="${ns}"/>
+  <xacro:mir prefix="${prefix}" ns="${ns}"/>
   <xacro:diff_controller_plugin_gazebo prefix="${prefix}" ns="${ns}"
     left_wheel_joint="${prefix}left_wheel_joint"
     right_wheel_joint="${prefix}right_wheel_joint"
-    wheel_separation="${2*mir_100_act_wheel_dy}"
-    wheel_radius="${mir_100_act_wheel_radius}"/>
+    wheel_separation="${2*mir_act_wheel_dy}"
+    wheel_radius="${mir_act_wheel_radius}"/>
 </robot>

Commit message: URDF: Make wheels black
This increases the contrast for the MiR 250 robot.

File: mir_description/urdf/include/mir_v1.urdf.xacro (robot description, xacro)
@@ -45,5 +45,5 @@
           <cylinder radius="${mir_act_wheel_radius}" length="${mir_act_wheel_width}" />
         </geometry>
-        <xacro:insert_block name="material_dark_grey" />
+        <xacro:insert_block name="material_black" />
       </visual>
       <collision>
@@ -55,5 +55,5 @@
     </link>
     <gazebo reference="${prefix}${locationprefix}_wheel_link">
-      <material>Gazebo/DarkGrey</material>
+      <material>Gazebo/FlatBlack</material>
     </gazebo>
   </xacro:macro>
@@ -131,5 +131,5 @@
           <cylinder radius="${mir_caster_wheel_radius}" length="${mir_caster_wheel_width}" />
         </geometry>
-        <xacro:insert_block name="material_dark_grey" />
+        <xacro:insert_block name="material_black" />
       </visual>
       <collision>
@@ -141,5 +141,5 @@
     </link>
     <gazebo reference="${prefix}${locationprefix}_caster_wheel_link">
-      <material>Gazebo/DarkGrey</material>
+      <material>Gazebo/FlatBlack</material>
     </gazebo>
   </xacro:macro>

Commit message: WIP: Partially port "Add arg mir_type to launch files and urdfs"

File: mir_description/urdf/include/mir_v1.urdf.xacro (robot description, xacro)
@@ -1,4 +1,6 @@
 <?xml version="1.0"?>
 <robot xmlns:xacro="http://ros.org/wiki/xacro">
+  <xacro:arg name="mir_type" default="mir_100" />      <!-- The MiR variant. Can be "mir_100" or "mir_250" for now.-->
+  <xacro:property name="mir_type" value="$(arg mir_type)" />  <!-- necessary because args cannot be accessed inside ${} expressions -->
   <xacro:include filename="$(find mir_description)/urdf/include/common_properties.urdf.xacro" />
   <xacro:include filename="$(find mir_description)/urdf/include/imu.gazebo.urdf.xacro" />
@@ -158,5 +160,5 @@
         <origin xyz="${mir_act_wheel_dx} 0 0" rpy="0 0 0" />
         <geometry>
-          <mesh filename="package://mir_description/meshes/visual/mir_100_base.stl" />
+          <mesh filename="package://mir_description/meshes/visual/${mir_type}_base.stl" />
         </geometry>
         <xacro:insert_block name="material_white" />
@@ -165,5 +167,5 @@
         <origin xyz="${mir_act_wheel_dx} 0 0" rpy="0 0 0" />
         <geometry>
-          <mesh filename="package://mir_description/meshes/collision/mir_100_base.stl" />
+          <mesh filename="package://mir_description/meshes/collision/${mir_type}_base.stl" />
         </geometry>
       </collision>
